File: docs/Kicad/FilterDesign/Sallen-key topology low-pass.kicad_sch (KiCad schematic)
At the start: 10 parts, among them J5 Conn_01x02_Pin, U2 MCP6002-xMC

Commit message: Staged changes to be able to merge to main
Connections:
- net +3.3V renamed +5V
Changed lines of the file:
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@@
 			)
 		)
-		(property "Value" "+3.3V"
-			(at 109.22 49.53 0)
+		(property "Value" "+5V"
+			(at 111.76 53.3399 0)
 			(effects
 				(font
 					(size 1.27 1.27)
 				)
+				(justify left)
 			)
 		)
