File: docs/Kicad/FilterDesign/AktivtFilterSim/AktivtFilterSim.kicad_sch (KiCad schematic)
At the start: 12 parts, among them J1 Conn_01x02_Pin, J2 Conn_01x02_Pin, U1 TLV9062

Commit message: spi stresstest & Kicad stuff
Parts:
- removed U1: TLV9062, symbol Amplifier_Operational:TLV9062
- added U1, U2: MCP6001-OT, Package_TO_SOT_SMD:SOT-23-5, symbol Amplifier_Operational:MCP6001-OT
- added U3: TLV3501AIDBV, Package_TO_SOT_SMD:SOT-23-6, symbol Comparator:TLV3501AIDBV
- added V1: 1, symbol Simulation_SPICE:VDC
- added Vsaw1, Vtriangle1: VSIN, symbol Simulation_SPICE:VSIN
- R5: value 1M -> 100k
Connections:
- net +3.3V: now also U1.5 (V+), U2.5 (V+), U3.4 (V+), U3.6 (SHDN), V1.1
- net GND: now also U1.2 (V-), U2.2 (V-), U3.2 (V-), V1.2, Vsaw1.2, Vtriangle1.2
- net out1: now also U1.1, U1.4 (-)
- net out2: now also U2.1, U2.4 (-)
- net at C4.1, R4.2: now also U2.3 (+)
- net at C3.1, R2.2: now also U1.3 (+)
- new net out: U3.1 (-), U3.3 (+), Vsaw1.1, Vtriangle1.1
- new net outcomp: U3.5
Other:
- note added: "* 390 kHz triangle wave: 0 → 3.3V → 0V every 2.564 µs Vtriangle triangle 0 PWL(0 0 1.282u 3.3 2.564u 0) REPEAT FOREVER"
- note added: "* 50 Hz sawtooth rising from 0V to 3.3V in 20ms, then reset Vsaw saw 0 PWL(0 0 20m 3.3) REPEAT FOREVER"
- note added: ".tran 10n 1m uic"
- note removed: ".tran 10n 2m"

Commit message: Staged changes to be able to merge to main
Connections:
- net +3.3V: no longer V1.1
- new net +5V: V1.1
Changed lines of the file:
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@@
 			)
 		)
-		(property "Value" "+3.3V"
-			(at 69.85 64.77 0)
+		(property "Value" "+5V"
+			(at 72.39 68.5799 0)
 			(effects
 				(font
 					(size 1.27 1.27)
 				)
+				(justify left)
 			)
 		)
