File: docs/Kicad/FilterDesign/Comparator/Comparator.kicad_sch (KiCad schematic)
At the start: 4 parts, among them U1 TLV3501AIDBV

Commit message: Staged changes to be able to merge to main
Connections:
- net +3.3V: no longer V1.1
- new net +5V: V1.1
Changed lines of the file:
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@@
 			)
 		)
-		(property "Value" "+3.3V"
-			(at 111.76 38.1 0)
+		(property "Value" "+5V"
+			(at 114.3 41.9099 0)
 			(effects
 				(font
 					(size 1.27 1.27)
 				)
+				(justify left)
 			)
 		)
